File: keyboard.kicad_pcb (KiCad board)
At the start: 2 copper layers, 285 x 94.6 mm, 338 parts, among them IC1 ATMEGA32U4, J1 MINI, P1 CONN_1, P10 CONN_1, P11 CONN_1, P12 CONN_1, P13 CONN_1, P14 CONN_1, P15 CONN_1, P16 CONN_1, P17 CONN_1, P18 CONN_1, P19 CONN_1, P2 CONN_1, P20 CONN_1, P21 CONN_1, P22 CONN_1, P23 CONN_1, P24 CONN_1, P25 CONN_1, P26 CONN_1, P27 CONN_1, P28 CONN_1, P29 CONN_1, P3 CONN_1, P30 CONN_1, P31 CONN_1, P32 CONN_1, P33 CONN_1, P34 CONN_1, P35 CONN_1, P36 CONN_1, P37 CONN_1, P38 CONN_1, P39 CONN_1, P4 CONN_1, P40 CONN_1, P41 CONN_1, P42 CONN_1, P5 CONN_1, P6 CONN_1, P7 CONN_1, P8 CONN_1, P9 CONN_1, X1 ASX3F

Commit message: Incomplete layout with IO expanders only. Next will switch back to matrix.
Parts:
- removed D01, D02, D03, D04, D05, D06, D07, D08, D09, D10, D11, D12, D13, D14, D15, D16, D17, D18, D19, D21, D22, D23, D24, D26, D27, D28, D29, D30, D31, D32, D33, D34, D36, D37, D38, D39, D41, D42, D43, D44, D46, D47, D48, D49, D50, D51, D52, D53, D54, D55, D56, D57, D58, D59, D60, D61, D62, D63, D64, D65, D66, D67, D68, D69, D70: 1N4148, 0805:0805D
- removed DB02, DB04, DB041, DB06, DB07, DB09, DB11, DB14, DB16, DB17, DB19, DB21, DB22, DB23, DB24, DB26, DB27, DB28, DB29, DB30, DB301, DB302, DB31, DB32, DB33, DB34, DB36, DB37, DB38, DB39, DB41, DB42, DB43, DB44, DB46, DB47, DB48, DB49, DB50, DB51, DB52, DB53, DB54, DB56, DB57, DB58, DB59, DB61, DB62, DB63, DB66, DB661, DB67, DB68, DB681, DB682, DB69, DC1, DC2, DF10, DF11, DF20, DF201, DF3, DW1, DW2, DW3, DW4: LED, mx1a:MX1A-led_no3d
- removed DB05, DB051, DB10, DB101, DB102, DB15, DB151, DB55, DB551, DF21, DF211, DF22, DF221, DF23, DF231, DF232: LEDa, MX1A-led
- removed DC3: LED, MX1A-ledlock
- removed FID (x2): FIDUCIAL, hole:FIDUCIAL
- removed the G*** at (228.1, 147.6)
- removed the HOLE at (345.8, 121.1)
- removed the HOLE at (63.7, 121.1)
- removed the HOLE at (322.3, 92.5)
- removed the HOLE at (252.8, 149.8)
- removed the HOLE at (190.5, 111.6)
- removed IC1: ATMEGA32U4, tqfp:TQFP44
- removed J1: MINI, usb:67503
- removed MXST (x15): VAL**, mx1a:MXST
- removed MXWIRE (x9): VAL**, MX1A-wire
- removed P1, P10, P11, P12, P13, P14, P15, P16, P17, P18, P19, P2, P20, P21, P22, P23, P24, P25, P26, P27, P28, P29, P3, P30, P31, P32, P33, P34, P35, P36, P37, P38, P39, P4, P40, P41, P42, P5, P6, P7, P8, P9: CONN_1, pad
- removed R10, R11, R12, R13, R14, R15: R, res:resistor
- removed S0: DTSM-6, dtsm:KSEM31GLFS
- removed S031, S041, S0512, S09, S102, S301, S302, S602, S63, S641, S682, S692, S7012: MX1Aa, mx1a:MX1A_no3d
- removed S10, S15, S55, S60, S65, S66, S69: MX1A, mx1a:MX1A
- removed S681: MX1A, mx1a:MX1A_no3d
- removed X1: ASX3F, ndk:4-SMD
- added HOLE: VAL**, hole:PKRHC, F.Cu at (343.5, 121.3)
- added HOLE: VAL**, hole:PKRHC, F.Cu at (66.0, 121.3)
- added HOLE: VAL**, hole:PKRHC, F.Cu at (190.5, 111.6)
- added HOLE: VAL**, hole:PKRHC, F.Cu at (252.8, 149.8)
- added HOLE: VAL**, hole:PKRHC, F.Cu at (322.3, 92.5)
- added Q1: BSS138, TO_SOT_Packages_SMD:SOT-23, F.Cu at (227.0, 144.5)
- added Q2: BSS138, TO_SOT_Packages_SMD:SOT-23, F.Cu at (220.0, 144.5)
- added Q3: BSS138, TO_SOT_Packages_SMD:SOT-23, F.Cu at (213.8, 144.5)
- added TOF1: VL6180X, VL6180X:VL6180X, F.Cu at (131.1, 143.5)
- added TOF2: VL6180X, VL6180X:VL6180X, F.Cu at (255.0, 143.5)
- added U1: TCA9555, Housings_DFN_QFN:QFN-24_4x4mm_Pitch0.5mm, F.Cu at (101.6, 124.5)
- added U2: TCA9555, Housings_DFN_QFN:QFN-24_4x4mm_Pitch0.5mm, F.Cu at (198.1, 102.3)
- added U3: TCA9555, Housings_DFN_QFN:QFN-24_4x4mm_Pitch0.5mm, F.Cu at (213.4, 102.2)
- added U4: TCA9555, Housings_DFN_QFN:QFN-24_4x4mm_Pitch0.5mm, F.Cu at (307.3, 114.3)
- added U5: FEATHER, feather:Feather-SMD, B.Cu at (226.7, 146.1)
- added U6: MIC5225_2.8V, TO_SOT_Packages_SMD:SOT-23-5, F.Cu at (235.5, 148.0)
- C1, C2: value 22p -> .1uF; footprint 0805:0805C -> Capacitors_SMD:C_0603_HandSoldering; moved to F.Cu
- C3: value 1u -> 0.1uF; footprint 0805:0805C -> Capacitors_SMD:C_0603_HandSoldering; moved to F.Cu
- C4, C5, C6: value 100n -> 0.1uF; footprint 0805:0805C -> Capacitors_SMD:C_0603_HandSoldering; moved to F.Cu
- C7: value 100n -> 10uF; footprint 0805:0805C -> Capacitors_SMD:C_0603_HandSoldering; moved to F.Cu
- C8: value 1u -> 10uF; footprint 0805:0805C -> Capacitors_SMD:C_0603_HandSoldering; moved to F.Cu
- R1, R2: value 22 -> 10K; footprint 0805:0805R -> Resistors_SMD:R_0603_HandSoldering; moved to F.Cu
- R3: value 10k -> 10K; footprint 0805:0805R -> Resistors_SMD:R_0603_HandSoldering; moved to F.Cu
- R4: value 300 -> 47K; footprint res:resistor -> Resistors_SMD:R_0603_HandSoldering; moved to F.Cu
- R5: value 10k -> 47K; footprint 0805:0805R -> Resistors_SMD:R_0603_HandSoldering; moved to F.Cu
- R6, R7, R8: value R -> 10K; footprint res:resistor -> Resistors_SMD:R_0603_HandSoldering; moved to F.Cu
- R9: value R -> 47K; footprint res:resistor -> Resistors_SMD:R_0603_HandSoldering; moved to F.Cu
- S1: renamed from S01; footprint mx1a:MX1A -> mx1a:MX1A-1U
- S11, S12, S13, S14, S16, S17, S18, S19, S21, S22, S23, S24, S26, S27, S28, S29, S31, S32, S33, S34, S36, S37, S38, S39, S41, S42, S43, S44, S46, S47, S48, S49, S51, S52, S53, S54, S56, S57, S58, S59, S61, S62, S70: footprint mx1a:MX1A -> mx1a:MX1A-1U
- S151, S50, S552, S601, S6512, S661: value MX1Aa -> MX1A; footprint mx1a:MX1A_no3d -> mx1a:MX1A-1U
- S6: renamed from S06; footprint mx1a:MX1A -> mx1a:MX1A-1U
- S7: renamed from S07; footprint mx1a:MX1A -> mx1a:MX1A-1U
- S8: renamed from S08; footprint mx1a:MX1A -> mx1a:MX1A-1U
- caps1: renamed from S03; footprint mx1a:MX1A -> mx1a:MX1A-1.75U
- ctl1: renamed from S05; footprint mx1a:MX1A -> mx1a:MX1A-1.25U
- enter1: renamed from S68; footprint mx1a:MX1A -> mx1a:MX1A-2.25U
- lshift1: renamed from S04; footprint mx1a:MX1A -> mx1a:MX1A-2.25U
- ltab1: renamed from S02; footprint mx1a:MX1A -> mx1a:MX1A-1.5U
- pipe1: renamed from S67; footprint mx1a:MX1A -> mx1a:MX1A-1.5U
- rshift1: renamed from S691; value MX1Aa -> MX1A; footprint mx1a:MX1A_no3d -> mx1a:MX1A-1.75U
- spacebar1: renamed from S30; footprint mx1a:MX1A -> mx1a:MX1A-6.25U
- up1: renamed from S64; footprint mx1a:MX1A_no3d -> mx1a:MX1A-1U
- win1: renamed from S101; value MX1Aa -> MX1A; footprint mx1a:MX1A_no3d -> mx1a:MX1A-1.25U
- moved C8 173.0 mm to (235.5, 144.5)
- moved R9 161.1 mm to (254.8, 139.2), turned to 180 degrees
- moved R2 150.7 mm to (217.0, 144.5), turned to 270 degrees
- moved R1 146.8 mm to (210.5, 144.5), turned to 270 degrees
- moved C6 139.8 mm to (306.8, 118.7), turned to 0 degrees
- moved R6 108.5 mm to (227.0, 140.0), turned to 0 degrees
- moved R8 88.5 mm to (216.3, 140.0), turned to 180 degrees
- moved R7 87.6 mm to (222.0, 140.0), turned to 0 degrees
- moved C2 83.5 mm to (258.5, 142.7), turned to 270 degrees
- moved R3 82.1 mm to (224.0, 144.5), turned to 270 degrees
- moved C4 72.2 mm to (203.0, 102.0), turned to 90 degrees
- moved C5 68.9 mm to (209.5, 103.5), turned to 270 degrees
- moved C3 65.2 mm to (106.3, 124.7), turned to 90 degrees
- moved C7 64.1 mm to (235.5, 151.5), turned to 0 degrees
- moved C1 40.2 mm to (135.8, 142.7), turned to 270 degrees
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Connections:
- C1 pad 1: N-000001 -> GND
- C1 pad 2: GND -> VDD
- C2 pad 1: N-000012 -> GND
- C2 pad 2: GND -> VDD
- C3 pad 1: N-000011 -> VCC
- C7 pad 1: VCC -> GND
- C7 pad 2: GND -> VCC
- C8 pad 1: VCC -> GND
- C8 pad 2: GND -> VDD
- R1 pad 1: N-000010 -> VDD
- R1 pad 2: N-000008 -> /TOF2_CE_28
- R2 pad 1: N-000009 -> VDD
- R2 pad 2: N-000007 -> /TOF_SDA_28
- R3 pad 1: N-000006 -> VDD
- R3 pad 2: GND -> /TOF_SCL_28
- R4 pad 1: N-000133 -> VDD
- R4 pad 2: /Matrix/CAPS_LED -> Net-(R4-Pad2)
- R5 pad 1: VCC -> VDD
- R5 pad 2: /~RES~ -> Net-(R5-Pad2)
- R6 pad 1: /GPIO0 -> VCC
- R6 pad 2: N-000004 -> /TOF_SCL
- R7 pad 1: /GPIO0 -> VCC
- R7 pad 2: N-000003 -> /TOF_SDA
- R8 pad 1: /GPIO0 -> VCC
- R8 pad 2: N-000002 -> /TOF2_CE
- R9 pad 1: /GPIO0 -> VDD
- S1 pad 1: /Matrix/row1 -> GND
- S11 pad 1: /Matrix/row1 -> Net-(S11-Pad1)
- S11 pad 2: N-000108 -> GND
- S12 pad 1: /Matrix/row2 -> Net-(S12-Pad1)
- S12 pad 2: N-000097 -> GND
- S13 pad 1: /Matrix/row3 -> Net-(S13-Pad1)
- S13 pad 2: N-000101 -> GND
- S14 pad 1: /Matrix/row4 -> Net-(S14-Pad1)
- S14 pad 2: N-000103 -> GND
- S151 pad 1: /Matrix/row5 -> Net-(S151-Pad1)
- S151 pad 2: N-000093 -> GND
- S16 pad 1: /Matrix/row1 -> Net-(S16-Pad1)
- S16 pad 2: N-000070 -> GND
- S17 pad 1: /Matrix/row2 -> Net-(S17-Pad1)
- S17 pad 2: N-000074 -> GND
- S18 pad 1: /Matrix/row3 -> Net-(S18-Pad1)
- S18 pad 2: N-000075 -> GND
- S19 pad 1: /Matrix/row4 -> Net-(S19-Pad1)
- S19 pad 2: N-000076 -> GND
- S21 pad 1: /Matrix/row1 -> Net-(S21-Pad1)
- S21 pad 2: N-000086 -> GND
- S22 pad 1: /Matrix/row2 -> Net-(S22-Pad1)
- S22 pad 2: N-000080 -> GND
- S23 pad 1: /Matrix/row3 -> Net-(S23-Pad1)
- S23 pad 2: N-000085 -> GND
- S24 pad 1: /Matrix/row4 -> Net-(S24-Pad1)
- S24 pad 2: N-000124 -> GND
- S26 pad 1: /Matrix/row1 -> Net-(S26-Pad1)
- S26 pad 2: N-000106 -> GND
- S27 pad 1: /Matrix/row2 -> Net-(S27-Pad1)
- S27 pad 2: N-000071 -> GND
- S28 pad 1: /Matrix/row3 -> Net-(S28-Pad1)
- S28 pad 2: N-000072 -> GND
- S29 pad 1: /Matrix/row4 -> Net-(S29-Pad1)
- S29 pad 2: N-000073 -> GND
- S31 pad 1: /Matrix/row1 -> Net-(S31-Pad1)
- S31 pad 2: N-000087 -> GND
- S32 pad 1: /Matrix/row2 -> Net-(S32-Pad1)
- S32 pad 2: N-000090 -> GND
- S33 pad 1: /Matrix/row3 -> Net-(S33-Pad1)
- S33 pad 2: N-000089 -> GND
- S34 pad 1: /Matrix/row4 -> Net-(S34-Pad1)
- S34 pad 2: N-000125 -> GND
- S36 pad 1: /Matrix/row1 -> Net-(S36-Pad1)
- S36 pad 2: N-000091 -> GND
- S37 pad 1: /Matrix/row2 -> Net-(S37-Pad1)
- S37 pad 2: N-000078 -> GND
- S38 pad 1: /Matrix/row3 -> Net-(S38-Pad1)
- S38 pad 2: N-000079 -> GND
- S39 pad 1: /Matrix/row4 -> Net-(S39-Pad1)
- S39 pad 2: N-000126 -> GND
- S41 pad 1: /Matrix/row1 -> Net-(S41-Pad1)
- S41 pad 2: N-000077 -> GND
- S42 pad 1: /Matrix/row2 -> Net-(S42-Pad1)
- S42 pad 2: N-000082 -> GND
- S43 pad 1: /Matrix/row3 -> Net-(S43-Pad1)
- S43 pad 2: N-000081 -> GND
- S44 pad 1: /Matrix/row4 -> Net-(S44-Pad1)
- S44 pad 2: N-000116 -> GND
- S46 pad 1: /Matrix/row1 -> Net-(S46-Pad1)
- S46 pad 2: N-000083 -> GND
- S47 pad 1: /Matrix/row2 -> Net-(S47-Pad1)
- S47 pad 2: N-000084 -> GND
- S48 pad 1: /Matrix/row3 -> Net-(S48-Pad1)
- S48 pad 2: N-000115 -> GND
- S49 pad 1: /Matrix/row4 -> Net-(S49-Pad1)
- S49 pad 2: N-000118 -> GND
- S50 pad 1: /Matrix/row5 -> Net-(S50-Pad1)
- S50 pad 2: N-000109 -> GND
- S51 pad 1: /Matrix/row1 -> Net-(S51-Pad1)
- S51 pad 2: N-000095 -> GND
- S52 pad 1: /Matrix/row2 -> Net-(S52-Pad1)
- S52 pad 2: N-000114 -> GND
- S53 pad 1: /Matrix/row3 -> Net-(S53-Pad1)
- S53 pad 2: N-000112 -> GND
- S54 pad 1: /Matrix/row4 -> Net-(S54-Pad1)
- S54 pad 2: N-000119 -> GND
- S552 pad 1: /Matrix/row5 -> Net-(S552-Pad1)
- S552 pad 2: N-000094 -> GND
- S56 pad 1: /Matrix/row1 -> Net-(S56-Pad1)
- S56 pad 2: N-000123 -> GND
- S57 pad 1: /Matrix/row2 -> Net-(S57-Pad1)
- S57 pad 2: N-000121 -> GND
- S58 pad 1: /Matrix/row3 -> Net-(S58-Pad1)
- S58 pad 2: N-000111 -> GND
- S59 pad 1: /Matrix/row4 -> Net-(S59-Pad1)
- S59 pad 2: N-000120 -> GND
- S6 pad 1: /Matrix/row1 -> Net-(S6-Pad1)
- S6 pad 2: N-000107 -> GND
- S601 pad 1: /Matrix/row5 -> Net-(S601-Pad1)
- S601 pad 2: N-000134 -> GND
- S61 pad 1: /Matrix/row1 -> Net-(S61-Pad1)
- S61 pad 2: N-000122 -> GND
- S62 pad 1: /Matrix/row2 -> Net-(S62-Pad1)
- S62 pad 2: N-000117 -> GND
- S6512 pad 1: /Matrix/row5 -> Net-(S6512-Pad1)
- S6512 pad 2: N-000096 -> GND
- S661 pad 1: /Matrix/row1 -> Net-(S661-Pad1)
- S661 pad 2: N-000135 -> GND
- S7 pad 1: /Matrix/row2 -> Net-(S7-Pad1)
- S7 pad 2: N-000099 -> GND
- S70 pad 1: /Matrix/row5 -> Net-(S70-Pad1)
- S70 pad 2: N-000104 -> GND
- S8 pad 1: /Matrix/row3 -> Net-(S8-Pad1)
- S8 pad 2: N-000100 -> GND
- caps1 pad 1: /Matrix/row3 -> Net-(U1-Pad13)
- caps1 pad 2: N-000105 -> GND
- ctl1 pad 1: /Matrix/row5 -> Net-(U1-Pad15)
- ctl1 pad 2: N-000092 -> GND
- enter1 pad 1: /Matrix/row3 -> Net-(U4-Pad10)
- enter1 pad 2: N-000127 -> GND
- lshift1 pad 1: /Matrix/row4 -> Net-(U1-Pad14)
- lshift1 pad 2: N-000130 -> GND
- ltab1 pad 1: /Matrix/row2 -> Net-(U1-Pad12)
- ltab1 pad 2: N-000098 -> GND
- pipe1 pad 1: /Matrix/row2 -> Net-(U4-Pad11)
- pipe1 pad 2: N-000113 -> GND
- rshift1 pad 2: /Matrix/row4 -> GND
- spacebar1 pad 1: /Matrix/row5 -> Net-(U2-Pad17)
- spacebar1 pad 2: N-000129 -> GND
- up1 pad 2: /Matrix/row4 -> GND
- win1 pad 1: /Matrix/row5 -> Net-(U1-Pad16)
- win1 pad 2: N-000128 -> GND
Routing:
- net VCC: track 709.9 -> 5.39 mm, vias 10 -> 0
- net GND: track 718.3 -> 37.1 mm, vias 41 -> 7
- net /Leds/lrow5: track 586.3 -> 0.00 mm, vias 9 -> 0
- net /Matrix/row5: track 485.3 -> 0.00 mm, vias 2 -> 0
- net /GPIO3: track 466.7 -> 0.00 mm, vias 8 -> 0
- net /Matrix/row1: track 450.6 -> 0.00 mm, vias 2 -> 0
- net /Matrix/row4: track 404.3 -> 0.00 mm, vias 3 -> 0
- net /Leds/lrow4: track 402.9 -> 0.00 mm, vias 5 -> 0
- net /GPIO1: track 398.3 -> 0.00 mm, vias 4 -> 0
- net /Matrix/row3: track 388.6 -> 0.00 mm, vias 5 -> 0
- net /Matrix/row2: track 382.7 -> 0.00 mm, vias 3 -> 0
- net /GPIO2: track 372.2 -> 0.00 mm, vias 6 -> 0
- net /Matrix/col14: track 339.3 -> 0.00 mm, vias 5 -> 0
- net /Leds/lrow2: track 329.4 -> 0.00 mm, vias 1 -> 0
- net /GPIO0: track 291.9 -> 0.00 mm, vias 5 -> 0
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Other:
- board text removed: "0"
- board text removed: "1"
- board text removed: "2"
- board text removed: "3"
- board text removed: "A"
- board text removed: "GPIO"
- board text removed: "R1"
- board text removed: "R2"
- board text removed: "R3"
- board text removed: "R4"
- board text removed: "R5"
- board text removed: "W"
- board text removed: "http://gh60.info"
- board text removed: "top routing path Ø 2mm"
- board text removed: "v-score on left side"
- board text removed: "v-score on right side"

Commit message: Switch to a matrix. Not done yet because feather needs to move.
Parts:
- removed C3, C4, C5, C6: 0.1uF, Capacitors_SMD:C_0603_HandSoldering
- removed U3, U4: TCA9555, Housings_DFN_QFN:QFN-24_4x4mm_Pitch0.5mm
- added D1: 1N4148, 0805:0805D, F.Cu at (80.8, 68.7)
- added D10: 1N4148, 0805:0805D, F.Cu at (107.5, 145.0)
- added D11: 1N4148, 0805:0805D, F.Cu at (119.0, 69.0)
- added D12: 1N4148, 0805:0805D, F.Cu at (128.5, 87.7)
- added D13: 1N4148, 0805:0805D, F.Cu at (133.3, 107.0)
- added D14: 1N4148, 0805:0805D, F.Cu at (123.8, 125.7)
- added D15: 1N4148, 0805:0805D, F.Cu at (117.0, 141.5)
- added D16: 1N4148, 0805:0805D, F.Cu at (138.0, 69.0)
- added D17: 1N4148, 0805:0805D, F.Cu at (147.5, 88.0)
- added D18: 1N4148, 0805:0805D, F.Cu at (152.3, 107.0)
- added D19: 1N4148, 0805:0805D, F.Cu at (142.8, 126.0)
- added D2: 1N4148, 0805:0805D, F.Cu at (87.5, 85.7)
- added D21: 1N4148, 0805:0805D, F.Cu at (157.3, 68.7)
- added D22: 1N4148, 0805:0805D, F.Cu at (166.8, 87.7)
- added D23: 1N4148, 0805:0805D, F.Cu at (171.5, 106.7)
- added D24: 1N4148, 0805:0805D, F.Cu at (161.8, 126.0)
- added D26: 1N4148, 0805:0805D, F.Cu at (176.3, 68.7)
- added D27: 1N4148, 0805:0805D, F.Cu at (185.8, 87.7)
- added D28: 1N4148, 0805:0805D, F.Cu at (190.5, 104.2)
- added D29: 1N4148, 0805:0805D, F.Cu at (181.0, 126.0)
- added D3: 1N4148, 0805:0805D, F.Cu at (88.0, 107.0)
- added D30: 1N4148, 0805:0805D, F.Cu at (188.8, 140.2)
- added D31: 1N4148, 0805:0805D, F.Cu at (195.3, 69.0)
- added D32: 1N4148, 0805:0805D, F.Cu at (204.8, 87.7)
- added D33: 1N4148, 0805:0805D, F.Cu at (209.5, 107.0)
- added D34: 1N4148, 0805:0805D, F.Cu at (200.0, 126.0)
- added D36: 1N4148, 0805:0805D, F.Cu at (214.0, 69.0)
- added D37: 1N4148, 0805:0805D, F.Cu at (223.8, 88.2)
- added D38: 1N4148, 0805:0805D, F.Cu at (228.5, 107.0)
- added D39: 1N4148, 0805:0805D, F.Cu at (219.0, 126.0)
- added D4: 1N4148, 0805:0805D, F.Cu at (93.0, 120.0)
- added D41: 1N4148, 0805:0805D, F.Cu at (233.2, 68.7)
- added D42: 1N4148, 0805:0805D, F.Cu at (242.8, 88.2)
- added D43: 1N4148, 0805:0805D, F.Cu at (247.8, 107.0)
- added D44: 1N4148, 0805:0805D, F.Cu at (238.0, 126.0)
- added D46: 1N4148, 0805:0805D, F.Cu at (252.3, 69.0)
- added D47: 1N4148, 0805:0805D, F.Cu at (262.0, 88.2)
- added D48: 1N4148, 0805:0805D, F.Cu at (266.8, 107.0)
- added D49: 1N4148, 0805:0805D, F.Cu at (257.3, 126.0)
- added D5: 1N4148, 0805:0805D, F.Cu at (83.6, 145.5)
- added D50: 1N4148, 0805:0805D, F.Cu at (328.8, 67.2)
- added D51: 1N4148, 0805:0805D, F.Cu at (271.5, 68.7)
- added D52: 1N4148, 0805:0805D, F.Cu at (280.8, 88.0)
- added D53: 1N4148, 0805:0805D, F.Cu at (285.8, 107.0)
- added D54: 1N4148, 0805:0805D, F.Cu at (276.3, 126.0)
- added D55: 1N4148, 0805:0805D, F.Cu at (276.3, 145.0)
- added D56: 1N4148, 0805:0805D, F.Cu at (290.5, 68.7)
- added D57: 1N4148, 0805:0805D, F.Cu at (300.0, 87.7)
- added D58: 1N4148, 0805:0805D, F.Cu at (305.0, 107.0)
- added D59: 1N4148, 0805:0805D, F.Cu at (295.3, 126.0)
- added D6: 1N4148, 0805:0805D, F.Cu at (99.8, 68.7)
- added D60: 1N4148, 0805:0805D, F.Cu at (295.3, 145.0)
- added D61: 1N4148, 0805:0805D, F.Cu at (309.5, 70.0)
- added D62: 1N4148, 0805:0805D, F.Cu at (309.5, 81.2)
- added D64: 1N4148, 0805:0805D, F.Cu at (314.0, 126.0)
- added D65: 1N4148, 0805:0805D, F.Cu at (314.3, 145.0)
- added D66: 1N4148, 0805:0805D, F.Cu at (309.5, 77.2)
- added D67: 1N4148, 0805:0805D, F.Cu at (322.7, 98.5)
- added D68: 1N4148, 0805:0805D, F.Cu at (322.8, 102.5)
- added D69: 1N4148, 0805:0805D, F.Cu at (319.3, 124.2)
- added D7: 1N4148, 0805:0805D, F.Cu at (109.5, 87.7)
- added D70: 1N4148, 0805:0805D, F.Cu at (333.3, 143.7)
- added D8: 1N4148, 0805:0805D, F.Cu at (114.1, 107.0)
- S8: footprint mx1a:MX1A-1U -> MX1A-1U
- S_caps1: renamed from caps1; footprint mx1a:MX1A-1.75U -> MX1A-1.75U
- S_tab1: renamed from ltab1; footprint mx1a:MX1A-1.5U -> MX1A-1.5U
- U1, U2: value TCA9555 -> 74HC595; footprint Housings_DFN_QFN:QFN-24_4x4mm_Pitch0.5mm -> Housings_SSOP:TSSOP-16_4.4x5mm_Pitch0.65mm
- spacebar1: footprint mx1a:MX1A-6.25U -> MX1A-6.25U
- moved U5 67.9 mm to (158.8, 146.0)
- moved U1 59.7 mm to (155.8, 149.5), turned to 0 degrees
- moved U2 53.3 mm to (173.3, 149.5), turned to 180 degrees
- moved R8 17.5 mm to (227.0, 153.7), turned to 0 degrees
- moved Q3 14.4 mm to (226.8, 150.7)
- moved R1 14.3 mm to (223.5, 150.5)
- renumbered up1 to S64, enter1 to S_enter1, lshift1 to S_lshift1, ctl1 to S_mod1, win1 to S_mod2, rshift1 to S_rshift1, pipe1 to S_slash1, S151 to Smod3
Connections:
- S1 pad 1: GND -> /ROW1
- S1 pad 2: Net-(S1-Pad2) -> Net-(D1-Pad2)
- S11 pad 1: Net-(S11-Pad1) -> /ROW1
- S11 pad 2: GND -> Net-(D11-Pad2)
- S12 pad 1: Net-(S12-Pad1) -> /ROW2
- S12 pad 2: GND -> Net-(D12-Pad2)
- S13 pad 1: Net-(S13-Pad1) -> /ROW3
- S13 pad 2: GND -> Net-(D13-Pad2)
- S14 pad 1: Net-(S14-Pad1) -> /ROW4
- S14 pad 2: GND -> Net-(D14-Pad2)
- S16 pad 1: Net-(S16-Pad1) -> /ROW1
- S16 pad 2: GND -> Net-(D16-Pad2)
- S17 pad 1: Net-(S17-Pad1) -> /ROW2
- S17 pad 2: GND -> Net-(D17-Pad2)
- S18 pad 1: Net-(S18-Pad1) -> /ROW3
- S18 pad 2: GND -> Net-(D18-Pad2)
- S19 pad 1: Net-(S19-Pad1) -> /ROW4
- S19 pad 2: GND -> Net-(D19-Pad2)
- S21 pad 1: Net-(S21-Pad1) -> /ROW1
- S21 pad 2: GND -> Net-(D21-Pad2)
- S22 pad 1: Net-(S22-Pad1) -> /ROW2
- S22 pad 2: GND -> Net-(D22-Pad2)
- S23 pad 1: Net-(S23-Pad1) -> /ROW3
- S23 pad 2: GND -> Net-(D23-Pad2)
- S24 pad 1: Net-(S24-Pad1) -> /ROW4
- S24 pad 2: GND -> Net-(D24-Pad2)
- S26 pad 1: Net-(S26-Pad1) -> /ROW1
- S26 pad 2: GND -> Net-(D26-Pad2)
- S27 pad 1: Net-(S27-Pad1) -> /ROW2
- S27 pad 2: GND -> Net-(D27-Pad2)
- S28 pad 1: Net-(S28-Pad1) -> /ROW3
- S28 pad 2: GND -> Net-(D28-Pad2)
- S29 pad 1: Net-(S29-Pad1) -> /ROW4
- S29 pad 2: GND -> Net-(D29-Pad2)
- S31 pad 1: Net-(S31-Pad1) -> /ROW1
- S31 pad 2: GND -> Net-(D31-Pad2)
- S32 pad 1: Net-(S32-Pad1) -> /ROW2
- S32 pad 2: GND -> Net-(D32-Pad2)
- S33 pad 1: Net-(S33-Pad1) -> /ROW3
- S33 pad 2: GND -> Net-(D33-Pad2)
- S34 pad 1: Net-(S34-Pad1) -> /ROW4
- S34 pad 2: GND -> Net-(D34-Pad2)
- S36 pad 1: Net-(S36-Pad1) -> /ROW1
- S36 pad 2: GND -> Net-(D36-Pad2)
- S37 pad 1: Net-(S37-Pad1) -> /ROW2
- S37 pad 2: GND -> Net-(D37-Pad2)
- S38 pad 1: Net-(S38-Pad1) -> /ROW3
- S38 pad 2: GND -> Net-(D38-Pad2)
- S39 pad 1: Net-(S39-Pad1) -> /ROW4
- S39 pad 2: GND -> Net-(D39-Pad2)
- S41 pad 1: Net-(S41-Pad1) -> /ROW1
- S41 pad 2: GND -> Net-(D41-Pad2)
- S42 pad 1: Net-(S42-Pad1) -> /ROW2
- S42 pad 2: GND -> Net-(D42-Pad2)
- S43 pad 1: Net-(S43-Pad1) -> /ROW3
- S43 pad 2: GND -> Net-(D43-Pad2)
- S44 pad 1: Net-(S44-Pad1) -> /ROW4
- S44 pad 2: GND -> Net-(D44-Pad2)
- S46 pad 1: Net-(S46-Pad1) -> /ROW1
- S46 pad 2: GND -> Net-(D46-Pad2)
- S47 pad 1: Net-(S47-Pad1) -> /ROW2
- S47 pad 2: GND -> Net-(D47-Pad2)
- S48 pad 1: Net-(S48-Pad1) -> /ROW3
- S48 pad 2: GND -> Net-(D48-Pad2)
- S49 pad 1: Net-(S49-Pad1) -> /ROW4
- S49 pad 2: GND -> Net-(D49-Pad2)
- S50 pad 1: Net-(S50-Pad1) -> /ROW1
- S50 pad 2: GND -> Net-(D50-Pad2)
- S51 pad 1: Net-(S51-Pad1) -> /ROW1
- S51 pad 2: GND -> Net-(D51-Pad2)
- S52 pad 1: Net-(S52-Pad1) -> /ROW2
- S52 pad 2: GND -> Net-(D52-Pad2)
- S53 pad 1: Net-(S53-Pad1) -> /ROW3
- S53 pad 2: GND -> Net-(D53-Pad2)
- S54 pad 1: Net-(S54-Pad1) -> /ROW4
- S54 pad 2: GND -> Net-(D54-Pad2)
- S552 pad 1: Net-(S552-Pad1) -> /ROW5
- S552 pad 2: GND -> Net-(D55-Pad2)
- S56 pad 1: Net-(S56-Pad1) -> /ROW1
- S56 pad 2: GND -> Net-(D56-Pad2)
- S57 pad 1: Net-(S57-Pad1) -> /ROW2
- S57 pad 2: GND -> Net-(D57-Pad2)
- S58 pad 1: Net-(S58-Pad1) -> /ROW3
- S58 pad 2: GND -> Net-(D58-Pad2)
- S59 pad 1: Net-(S59-Pad1) -> /ROW4
- S59 pad 2: GND -> Net-(D59-Pad2)
- S6 pad 1: Net-(S6-Pad1) -> /ROW1
- S6 pad 2: GND -> Net-(D6-Pad2)
- S601 pad 1: Net-(S601-Pad1) -> /ROW5
- S601 pad 2: GND -> Net-(D60-Pad2)
- S61 pad 1: Net-(S61-Pad1) -> /ROW2
- S61 pad 2: GND -> Net-(D61-Pad2)
- S62 pad 1: Net-(S62-Pad1) -> /ROW3
- S62 pad 2: GND -> Net-(D62-Pad2)
- S64 pad 1: Net-(U4-Pad5) -> /ROW4
- S64 pad 2: GND -> Net-(D64-Pad2)
- S6512 pad 1: Net-(S6512-Pad1) -> /ROW5
- S6512 pad 2: GND -> Net-(D65-Pad2)
- S661 pad 1: Net-(S661-Pad1) -> /ROW1
- S661 pad 2: GND -> Net-(D66-Pad2)
- S7 pad 1: Net-(S7-Pad1) -> /ROW2
- S7 pad 2: GND -> Net-(D7-Pad2)
- S70 pad 1: Net-(S70-Pad1) -> /ROW5
- S70 pad 2: GND -> Net-(D70-Pad2)
- S8 pad 1: Net-(S8-Pad1) -> /ROW3
- S8 pad 2: GND -> Net-(D8-Pad2)
- S_caps1 pad 1: Net-(U1-Pad13) -> /ROW3
- S_caps1 pad 2: GND -> Net-(D3-Pad2)
- S_enter1 pad 1: Net-(U4-Pad10) -> /ROW3
- S_enter1 pad 2: GND -> Net-(D68-Pad2)
- S_lshift1 pad 1: Net-(U1-Pad14) -> /ROW4
- S_lshift1 pad 2: GND -> Net-(D4-Pad2)
- S_mod1 pad 1: Net-(U1-Pad15) -> /ROW5
- S_mod1 pad 2: GND -> Net-(D5-Pad2)
- S_mod2 pad 1: Net-(U1-Pad16) -> /ROW5
- S_mod2 pad 2: GND -> Net-(D10-Pad2)
- S_rshift1 pad 1: Net-(U4-Pad8) -> /ROW4
- S_rshift1 pad 2: GND -> Net-(D69-Pad2)
- S_slash1 pad 1: Net-(U4-Pad11) -> /ROW2
- S_slash1 pad 2: GND -> Net-(D67-Pad2)
- S_tab1 pad 1: Net-(U1-Pad12) -> /ROW2
- S_tab1 pad 2: GND -> Net-(D2-Pad2)
- Smod3 pad 1: Net-(S151-Pad1) -> /ROW5
- Smod3 pad 2: GND -> Net-(D15-Pad2)
- TOF1 pad 11: Net-(TOF1-Pad11) -> (no net)
- TOF1 pad 2: Net-(TOF1-Pad2) -> (no net)
- TOF1 pad 3: Net-(TOF1-Pad3) -> (no net)
- TOF1 pad 7: Net-(TOF1-Pad7) -> (no net)
- TOF2 pad 11: Net-(TOF2-Pad11) -> (no net)
- TOF2 pad 2: Net-(TOF2-Pad2) -> (no net)
- TOF2 pad 3: Net-(TOF2-Pad3) -> (no net)
- TOF2 pad 7: Net-(TOF2-Pad7) -> (no net)
- U1 pad 1: Net-(S14-Pad1) -> /COL7
- U1 pad 10: Net-(S6-Pad1) -> VCC
- U1 pad 11: Net-(S1-Pad2) -> /COL_CLK
- U1 pad 12: Net-(U1-Pad12) -> /COL_CLK
- U1 pad 13: Net-(U1-Pad13) -> GND
- U1 pad 14: Net-(U1-Pad14) -> /COL_DATA
- U1 pad 15: Net-(U1-Pad15) -> /COL8
- U1 pad 16: Net-(U1-Pad16) -> VCC
- U1 pad 2: Net-(S19-Pad1) -> /COL6
- U1 pad 3: Net-(S18-Pad1) -> /COL5
- U1 pad 4: Net-(S13-Pad1) -> /COL4
- U1 pad 5: Net-(S12-Pad1) -> /COL3
- U1 pad 6: Net-(S11-Pad1) -> /COL2
- U1 pad 7: Net-(S8-Pad1) -> /COL1
- U1 pad 8: Net-(S7-Pad1) -> GND
- U1 pad 9: GND -> Net-(U1-Pad9)
- U2 pad 1: Net-(U2-Pad1) -> /COL14
- U2 pad 10: Net-(S17-Pad1) -> VCC
- U2 pad 11: Net-(S23-Pad1) -> /COL_CLK
- U2 pad 12: Net-(S28-Pad1) -> /COL_CLK
- U2 pad 13: Net-(S24-Pad1) -> GND
- U2 pad 14: Net-(S29-Pad1) -> Net-(U1-Pad9)
- U2 pad 15: Net-(S34-Pad1) -> (no net)
- U2 pad 16: Net-(S33-Pad1) -> VCC
- U2 pad 2: Net-(S31-Pad1) -> /COL13
- U2 pad 3: Net-(S32-Pad1) -> /COL12
- U2 pad 4: Net-(S26-Pad1) -> /COL11
- U2 pad 5: Net-(S21-Pad1) -> /COL10
- U2 pad 6: Net-(S16-Pad1) -> /COL9
- U2 pad 7: Net-(S27-Pad1) -> (no net)
- U2 pad 8: Net-(S22-Pad1) -> GND
- U2 pad 9: GND -> (no net)
- U5 pad 1: Net-(U5-Pad1) -> (no net)
- U5 pad 10: Net-(U5-Pad10) -> (no net)
- U5 pad 11: Net-(U5-Pad11) -> (no net)
- U5 pad 12: Net-(U5-Pad12) -> (no net)
- U5 pad 13: Net-(U5-Pad13) -> (no net)
- U5 pad 14: /INT3 -> (no net)
- U5 pad 15: /INT4 -> (no net)
- U5 pad 16: Net-(U5-Pad16) -> (no net)
- U5 pad 17: /KEYS_SDA -> /TOF_SDA
- U5 pad 18: /KEYS_SCL -> /TOF_SCL
- U5 pad 19: Net-(U5-Pad19) -> /COL_CLK
- U5 pad 20: /TOF2_CE -> /COL_DATA
- U5 pad 21: /INT1 -> /ROW1
- U5 pad 22: /INT2 -> /ROW2
- U5 pad 23: /TOF_SDA -> /ROW3
- U5 pad 24: Net-(U5-Pad24) -> /ROW4
- U5 pad 25: /TOF_SCL -> /ROW5
- U5 pad 26: Net-(U5-Pad26) -> (no net)
- U5 pad 27: Net-(U5-Pad27) -> (no net)
- U5 pad 28: Net-(U5-Pad28) -> (no net)
- U5 pad 3: Net-(U5-Pad3) -> (no net)
- U5 pad 5: Net-(U5-Pad5) -> (no net)
- U5 pad 6: Net-(U5-Pad6) -> /TOF2_CE
- U5 pad 7: Net-(U5-Pad7) -> (no net)
- U5 pad 8: Net-(U5-Pad8) -> (no net)
- U5 pad 9: Net-(U5-Pad9) -> (no net)
- U6 pad 4: Net-(U6-Pad4) -> (no net)
- spacebar1 pad 1: Net-(U2-Pad17) -> /ROW5
- spacebar1 pad 2: GND -> Net-(D30-Pad2)
Routing:
- net /ROW2: track 0.00 -> 290.9 mm, vias 0 -> 2
- net /ROW1: track 0.00 -> 271.3 mm
- net /ROW5: track 0.00 -> 270.8 mm, vias 0 -> 2
- net /ROW3: track 0.00 -> 268.7 mm
- net /COL14: track 0.00 -> 267.7 mm, vias 0 -> 4
- net /ROW4: track 0.00 -> 251.9 mm, vias 0 -> 1
- net /COL13: track 0.00 -> 231.3 mm, vias 0 -> 6
- net /COL12: track 0.00 -> 221.2 mm, vias 0 -> 8
- net /COL11: track 0.00 -> 204.6 mm, vias 0 -> 10
- net VCC: track 5.39 -> 185.6 mm, vias 0 -> 3
- net /TOF_SDA_28: track 2.06 -> 170.8 mm, vias 0 -> 7
- net /COL1: track 0.00 -> 166.8 mm, vias 0 -> 10
- net /COL8: track 0.00 -> 144.4 mm, vias 0 -> 10
- net /COL7: track 0.00 -> 143.4 mm, vias 0 -> 10
- net /COL2: track 0.00 -> 142.6 mm, vias 0 -> 10
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
Commit message: Working version with closer to correct NeoPixel footprint.
Parts:
- added C3: 0.1uF, Capacitors_SMD:C_0603_HandSoldering, F.Cu at (155.8, 144.2)
- added C4: 0.1uF, Capacitors_SMD:C_0603_HandSoldering, F.Cu at (167.3, 152.7)
- added C5: 0.1uF, Capacitors_SMD:C_0603_HandSoldering, F.Cu at (335.8, 151.0)
- added C6: 4.7uF, Capacitors_SMD:C_0603_HandSoldering, F.Cu at (134.1, 146.0)
- added C9: 4.7uF, Capacitors_SMD:C_0603_HandSoldering, F.Cu at (258.9, 145.5)
- added U3: SK6812, neopixel:SK6812, F.Cu at (340.7, 150.0)
- D1, D10, D11, D12, D13, D14, D15, D16, D17, D18, D19, D2, D21, D22, D23, D24, D26, D27, D28, D29, D3, D30, D31, D32, D33, D34, D36, D37, D38, D39, D4, D41, D42, D43, D44, D46, D47, D48, D49, D5, D50, D51, D52, D53, D54, D55, D56, D57, D58, D59, D6, D60, D61, D62, D64, D65, D66, D67, D68, D69, D7, D70, D8: footprint 0805:0805D -> Diodes_SMD:D_SOD-123
- S8: footprint MX1A-1U -> mx1a:MX1A-1U
- S_caps1: footprint MX1A-1.75U -> mx1a:MX1A-1.75U
- S_tab1: footprint MX1A-1.5U -> mx1a:MX1A-1.5U
- spacebar1: footprint MX1A-6.25U -> mx1a:MX1A-6.25U
- moved D50 3.26 mm to (328.5, 70.5), turned to 90 degrees
- moved R4 2.53 mm to (135.3, 148.8)
- moved D2 2.25 mm to (87.5, 83.5)
- moved D66 2.25 mm to (309.5, 75.0), turned to 90 degrees
- moved D69 2.12 mm to (320.8, 125.7), turned to 90 degrees
- moved D1 1.77 mm to (81.0, 70.5), turned to 90 degrees
- moved D21 1.75 mm to (157.3, 70.5), turned to 90 degrees
- moved D26 1.75 mm to (176.3, 70.5), turned to 90 degrees
- moved D41 1.75 mm to (233.2, 70.5), turned to 90 degrees
- moved D51 1.75 mm to (271.5, 70.5), turned to 90 degrees
- moved D56 1.75 mm to (290.5, 70.5), turned to 90 degrees
- moved D6 1.75 mm to (99.8, 70.5), turned to 90 degrees
- moved D4 1.58 mm to (91.5, 120.5)
- moved D36 1.52 mm to (214.3, 70.5), turned to 90 degrees
- moved D11 1.50 mm to (119.0, 70.5), turned to 90 degrees
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Connections:
- U1 pad 15: /COL8 -> (no net)
- U2 pad 7: (no net) -> /COL8
- U5 pad 19: /COL_CLK -> /ROW1
- U5 pad 20: /COL_DATA -> /ROW2
- U5 pad 21: /ROW1 -> /ROW3
- U5 pad 22: /ROW2 -> /ROW4
- U5 pad 23: /ROW3 -> /ROW5
- U5 pad 24: /ROW4 -> /COL_CLK
- U5 pad 25: /ROW5 -> /COL_DATA
- U5 pad 7: (no net) -> /NEOPIX
Routing:
- net /NEOPIX: track 0.00 -> 192.4 mm, vias 0 -> 1
- net VCC: track 185.6 -> 337.1 mm, vias 3 -> 18
- net /TOF_SCL_28: track 50.4 -> 173.4 mm, vias 2 -> 6
- net VDD: track 80.4 -> 192.2 mm, vias 2 -> 6
- net /COL10: track 70.4 -> 173.9 mm, vias 6 -> 8
- net /TOF_SDA: track 23.2 -> 110.1 mm
- net /TOF_SCL: track 24.2 -> 109.1 mm
- net /ROW1: track 271.3 -> 356.1 mm, vias 0 -> 5
- net /COL9: track 70.1 -> 149.8 mm
- net GND: track 62.8 -> 130.2 mm, vias 8 -> 10
- net /TOF2_CE: track 8.29 -> 72.6 mm, vias 1 -> 3
- net /ROW2: track 290.9 -> 342.8 mm, vias 2 -> 5
- net /COL_DATA: track 63.0 -> 14.4 mm, vias 3 -> 1
- net /ROW3: track 268.7 -> 303.2 mm, vias 0 -> 1
- net /COL_CLK: track 16.3 -> 37.4 mm, vias 0 -> 1
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Other:
- net class Default: clearance 0.2032 -> 0.1524
- net class POWER: clearance 0.2032 -> 0.1524
- rule trace_clearance: 0.2032 -> 0.1524
- board text added: "PCB design by komar007, jdcarpe & tannewt"
- board text removed: "+"
- board text removed: "-"
- board text removed: "CAPS"
- board text removed: "D"
- board text removed: "ESC"
- board text removed: "Fn"
- board text removed: "PCB design by komar007 & jdcarpe"
- board text removed: "Poker arrows"
- board text removed: "S"
- board text removed: "dedicated to the memory of SmallFry"
- board text removed: "expansion module"
